File: PCB_Design/HV_POWER_SUPPLY_newshape/HV_POWER_SUPPLY_NEWSHAPE.kicad_sch (KiCad schematic)
At the start: 54 parts, among them J1 Conn_01x02, J2 Conn_01x02, J5 Conn_01x02, Q2 DMN10H220L-7, U1 SN74LVC1G08DCKR_C5279048, U3 LTC6906IS6#TRPBF

Commit message: -Zone clearance =.5 -added via for SYS_5V -adjust ground via
Parts:
- D1: Package SOD-323 -> SOD-123
Changed lines of the file:
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@@
 			)
 		)
-		(property "Package" "SOD-323"
+		(property "Package" "SOD-123"
 			(at 22.86 46.99 0)
 			(effects
