File: PCB_Design/HV_POWER_SUPPLY_newshape/Sheet2.kicad_sch (KiCad schematic)
At the start: 29 parts, among them J3 Conn_01x02, J4 Conn_01x02, M1 AI-1223-TWT-5V-5-R, U2 LTC1540IMS8#PBF, U4 LTC6994CS6-1-TRMPBF, U5 LTC1441CS8#PBF

Commit message: -Zone clearance =.5 -added via for SYS_5V -adjust ground via
Parts:
- D11, D12: Package SOD-323 -> SOD-123
Changed lines of the file:
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@@
 			)
 		)
-		(property "Package" "SOD-323"
+		(property "Package" "SOD-123"
 			(at 83.82 78.74 0)
 			(effects
@@
 			)
 		)
-		(property "Package" "SOD-323"
+		(property "Package" "SOD-123"
 			(at 83.82 57.15 0)
 			(effects
